File: R2020Interface-RS485.brd (EAGLE design)
At the start: 76.2 x 50.8 mm, 73 parts, among them IC1 SN65176BDR, IC2 ATmega328-AU, IC3 RT8289, IC4 LM5010SD, J1 RS485, J10 R2020, J11 Index Feedback, J12 R2020 !CS, J13 R2020 MISO, J14 R2020 MOSI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

Commit message: foo
Parts:
- S1: device freetronics-master-v1:TACTILE_SWITCH_SMD_2PIN_TINY -> freetronics-luke:FSMSM
- moved S1 5.36 mm to (31.1, 3.14), turned to 180 degrees
- moved SY1 0.32 mm to (7.78, 1.75)
Connections:
- net !RESET: now also S1.1; no longer S1.2
- net GND: now also S1.2; no longer S1.1
Routing:
- net RXD: track 29.5 -> 28.0 mm
- net !RESET: track 38.5 -> 39.7 mm
Changed lines of the file:
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@@
 <text x="52.54625" y="33.9725" size="0.8128" layer="21" ratio="15">SCK</text>
 <text x="54.9275" y="33.9725" size="0.8128" layer="21" ratio="15">PWM</text>
-<text x="10.4775" y="2.06375" size="0.8128" layer="21" ratio="15">R2020 Servo Controller</text>
-<text x="12.065" y="0.635" size="0.8128" layer="21" ratio="15">Luke Weston, 2013</text>
-<text x="32.54375" y="3.81" size="0.8128" layer="21" ratio="15">Reset</text>
+<text x="9.8425" y="2.06375" size="0.8128" layer="21" ratio="15">R2020 Servo Controller</text>
+<text x="10.95375" y="0.79375" size="0.8128" layer="21" ratio="15">Luke Weston, 2013</text>
+<text x="29.36875" y="5.08" size="0.8128" layer="21" ratio="15">Reset</text>
 <text x="6.82625" y="47.14875" size="0.8128" layer="21" ratio="15">Power</text>
 <text x="74.93" y="32.0675" size="0.8128" layer="21" ratio="15" rot="SR270">INDEX</text>
@@
 <attribute name="VALUE" x="48.8315" y="29.8323" size="0.8128" layer="27" font="vector" ratio="15"/>
 </element>
-<element name="S1" library="freetronics-master-v1" package="TACTILE_SWITCH_SMD_2PIN_TINY" value="Reset" x="34.29" y="7.46125" smashed="yes" rot="R270"/>
 <element name="J7" library="freetronics-master-v1" package="1X05" value="Encoder" x="62.23" y="17.78" smashed="yes" rot="R90">
 <attribute name="NAME" x="63.58255" y="22.62505" size="0.8128" layer="25" ratio="15"/>
@@
 <attribute name="VALUE" x="37.05225" y="1.7018" size="0.8128" layer="27" font="vector" ratio="15"/>
 </element>
-<element name="SY1" library="SparkFun" package="OSHW-LOGO-S" value="OSHW-LOGOS" x="8.09625" y="1.74625"/>
+<element name="SY1" library="SparkFun" package="OSHW-LOGO-S" value="OSHW-LOGOS" x="7.77875" y="1.74625"/>
 <element name="LED3" library="freetronics-master-v1" package="LED-0603" value="Power" x="8.09625" y="46.51375" smashed="yes">
 <attribute name="PACKAGE" value="0603" x="8.09625" y="46.51375" size="0.8128" layer="27" ratio="15" display="off"/>
@@
 <attribute name="NAME" x="47.371" y="17.018" size="0.4064" layer="25" font="vector"/>
 <attribute name="VALUE" x="19.14525" y="13.48105" size="0.8128" layer="27" font="vector" ratio="15"/>
+</element>
+<element name="S1" library="freetronics-luke" package="FSMSM" value="Reset" x="31.115" y="3.1369" smashed="yes" rot="R180">
+<attribute name="PACKAGE" value="FSMSM" x="31.115" y="3.1369" size="1.778" layer="27" rot="R180" display="off"/>
+<attribute name="NAME" x="29.36875" y="6.0706" size="0.8128" layer="25" ratio="15"/>
+<attribute name="VALUE" x="29.36875" y="5.1181" size="0.8128" layer="27" ratio="15"/>
 </element>
 </elements>
@@
 </polygon>
 <contactref element="LED5" pad="C"/>
-<contactref element="S1" pad="1"/>
 <contactref element="IC4" pad="5"/>
 <contactref element="IC4" pad="PAD"/>
@@
 <contactref element="C1" pad="1"/>
 <via x="41.43375" y="11.7475" extent="1-16" drill="0.4"/>
+<contactref element="S1" pad="2"/>
 </signal>
 <signal name="+5V">
@@
 <contactref element="IC1" pad="1"/>
 <via x="43.02125" y="7.14375" extent="1-16" drill="0.4"/>
-<wire x1="43.02125" y1="7.14375" x2="37.30625" y2="7.14375" width="0.4064" layer="16"/>
-<wire x1="37.30625" y1="7.14375" x2="35.56" y2="8.89" width="0.4064" layer="16"/>
 <via x="31.115" y="6.985" extent="1-16" drill="0.4"/>
 <wire x1="31.115" y1="6.985" x2="23.54625" y2="6.985" width="0.4064" layer="1"/>
-<wire x1="45.56125" y1="7.14375" x2="43.02125" y2="7.14375" width="0.4064" layer="1"/>
-<wire x1="31.115" y1="6.985" x2="33.02" y2="8.89" width="0.4064" layer="16"/>
-<wire x1="33.02" y1="8.89" x2="35.56" y2="8.89" width="0.4064" layer="16"/>
+<wire x1="31.115" y1="6.985" x2="42.2275" y2="6.985" width="0.4064" layer="16"/>
+<wire x1="43.02125" y1="7.14375" x2="42.38625" y2="7.14375" width="0.4064" layer="16"/>
+<wire x1="42.38625" y1="7.14375" x2="42.2275" y2="6.985" width="0.4064" layer="16"/>
+<wire x1="43.02125" y1="7.14375" x2="45.56125" y2="7.14375" width="0.4064" layer="1"/>
 </signal>
 <signal name="MOSI">
@@
 <contactref element="J9" pad="5"/>
 <contactref element="R6" pad="1"/>
-<contactref element="S1" pad="2"/>
 <contactref element="C3" pad="1"/>
 <contactref element="C7" pad="2"/>
 <wire x1="38.1" y1="5.08" x2="38.1" y2="3.14325" width="0.508" layer="1"/>
-<wire x1="34.29" y1="5.41125" x2="36.49875" y2="5.41125" width="0.508" layer="1"/>
-<wire x1="36.49875" y1="5.41125" x2="36.83" y2="5.08" width="0.508" layer="1"/>
-<wire x1="36.83" y1="5.08" x2="38.1" y2="5.08" width="0.508" layer="1"/>
 <wire x1="41.04" y1="9.6774" x2="41.04" y2="8.655" width="0.508" layer="1"/>
 <wire x1="38.1" y1="5.08" x2="38.1" y2="5.715" width="0.508" layer="1"/>
@@
 <wire x1="29.845" y1="10.95375" x2="29.845" y2="6.985" width="0.3048" layer="16"/>
 <wire x1="29.845" y1="6.985" x2="31.75" y2="5.08" width="0.3048" layer="16"/>
-<wire x1="34.29" y1="5.41125" x2="33.03375" y2="5.41125" width="0.4064" layer="1"/>
-<wire x1="33.03375" y1="5.41125" x2="32.7025" y2="5.08" width="0.4064" layer="1"/>
-<wire x1="32.7025" y1="5.08" x2="31.75" y2="5.08" width="0.4064" layer="1"/>
 <via x="31.75" y="5.08" extent="1-16" drill="0.4"/>
 <wire x1="32.258" y1="17.907" x2="32.09925" y2="17.907" width="0.4064" layer="1"/>
@@
 <wire x1="29.05125" y1="20.955" x2="29.05125" y2="23.97125" width="0.4064" layer="1"/>
 <wire x1="29.05125" y1="23.97125" x2="30.48" y2="25.4" width="0.4064" layer="1"/>
+<contactref element="S1" pad="1"/>
+<wire x1="38.1" y1="3.14325" x2="35.71875" y2="3.14325" width="0.508" layer="1"/>
+<wire x1="35.71875" y1="3.14325" x2="35.7124" y2="3.1369" width="0.508" layer="1"/>
+<wire x1="31.75" y1="5.08" x2="31.75" y2="3.96875" width="0.508" layer="1"/>
+<wire x1="31.75" y1="3.96875" x2="32.58185" y2="3.1369" width="0.508" layer="1"/>
+<wire x1="35.7124" y1="3.1369" x2="32.58185" y2="3.1369" width="0.508" layer="1"/>
 </signal>
 <signal name="!R2020_CS">
@@
 </signal>
 </signals>
-<errors>
-</errors>
 </board>
 </drawing>
