File: R2020Interface-RS485.sch (EAGLE design)
At the start: 73 parts, among them IC1 SN65176BDR, IC2 ATmega328-AU, IC3 RT8289, IC4 LM5010SD, J1 RS485, J10 R2020, J11 Index Feedback, J12 R2020 !CS, J13 R2020 MISO, J14 R2020 MOSI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

Commit message: foo
Parts:
- S1: device freetronics-master-v1:TAC_SWITCH_2PIN -> freetronics-luke:FSMSM; PACKAGE (none) -> FSMSM
Connections:
- net !RESET: now also S1.1; no longer S1.S
- net GND: now also S1.2; no longer S1.P
Changed lines of the file:
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@@
 </part>
 <part name="U$46" library="freetronics-luke" deviceset="+5V" device=""/>
-<part name="S1" library="freetronics-master-v1" deviceset="TAC_SWITCH_2PIN" device="" value="Reset"/>
 <part name="U$47" library="freetronics-luke" deviceset="GND" device=""/>
 <part name="J7" library="freetronics-master-v1" deviceset="M05" device="PTH" value="Encoder"/>
@@
 <part name="R3" library="freetronics-master-v1" deviceset="RESISTOR" device="0603" value="120Ω">
 <attribute name="PACKAGE" value="0603"/>
+</part>
+<part name="S1" library="freetronics-luke" deviceset="FSMSM" device="" value="Reset">
+<attribute name="PACKAGE" value="FSMSM"/>
 </part>
 </parts>
@@
 </instance>
 <instance part="U$46" gate="G$1" x="228.6" y="137.16" rot="MR0"/>
-<instance part="S1" gate="1" x="215.9" y="236.22" smashed="yes" rot="R90">
-<attribute name="NAME" x="208.28" y="231.14" size="1.27" layer="95"/>
-<attribute name="VALUE" x="208.28" y="228.6" size="1.27" layer="96"/>
-</instance>
 <instance part="U$47" gate="G$1" x="215.9" y="226.06"/>
 <instance part="J7" gate="G$1" x="152.4" y="271.78" smashed="yes" rot="R180">
@@
 <attribute name="NAME" x="91.44" y="325.12" size="1.27" layer="95"/>
 <attribute name="VALUE" x="91.44" y="322.58" size="1.27" layer="96"/>
+</instance>
+<instance part="S1" gate="G$1" x="215.9" y="236.22" smashed="yes" rot="R270">
+<attribute name="PACKAGE" x="208.28" y="233.68" size="1.27" layer="96"/>
+<attribute name="NAME" x="208.28" y="238.76" size="1.27" layer="95"/>
+<attribute name="VALUE" x="208.28" y="236.22" size="1.27" layer="96"/>
 </instance>
 </instances>
@@
 </segment>
 <segment>
-<pinref part="S1" gate="1" pin="P"/>
 <pinref part="U$47" gate="G$1" pin="GND"/>
 <wire x1="215.9" y1="228.6" x2="215.9" y2="231.14" width="0.1524" layer="91"/>
+<pinref part="S1" gate="G$1" pin="2"/>
 </segment>
 <segment>
@@
 <junction x="215.9" y="251.46"/>
 <label x="208.28" y="251.714" size="1.27" layer="95"/>
-<pinref part="S1" gate="1" pin="S"/>
-<wire x1="215.9" y1="241.3" x2="215.9" y2="251.46" width="0.1524" layer="91"/>
+<wire x1="215.9" y1="241.3" x2="215.9" y2="248.92" width="0.1524" layer="91"/>
 <pinref part="C7" gate="G$1" pin="2"/>
-<wire x1="223.52" y1="238.76" x2="223.52" y2="243.84" width="0.1524" layer="91"/>
-<wire x1="223.52" y1="243.84" x2="215.9" y2="251.46" width="0.1524" layer="91"/>
-</segment>
-<segment>
+<wire x1="215.9" y1="248.92" x2="215.9" y2="251.46" width="0.1524" layer="91"/>
+<pinref part="S1" gate="G$1" pin="1"/>
+<wire x1="223.52" y1="238.76" x2="223.52" y2="241.3" width="0.1524" layer="91"/>
+<wire x1="223.52" y1="241.3" x2="215.9" y2="248.92" width="0.1524" layer="91"/>
+<junction x="215.9" y="248.92"/>
+</segment>
+<segment>
