File: R2020Interface.brd (EAGLE design)
At the start: 91.4 x 50.8 mm, 83 parts, among them IC1 ATmega328-AU, IC2 RT8289, IC3 LM5010SD, IC4 MCP2515-I/SO, IC5 MCP2551, J1 ISP, J10 Position feedback pot, J11 CAN Terminate, J12 AS5040, J13 Encoder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

Commit message: foo
Parts:
- moved JP2 15.2 mm to (71.1, 3.81)
- moved R16 9.44 mm to (71.8, 41.9)
- moved R17 9.03 mm to (74.3, 42.5), turned to 90 degrees
- moved C16 8.01 mm to (76.4, 42.5), turned to 270 degrees
- moved JP1 6.35 mm to (80.0, 47.0)
- moved J4 4.42 mm to (79.7, 30.8)
- moved R13 2.84 mm to (67.3, 40.6), turned to 90 degrees
- moved J10 2.54 mm to (69.8, 35.6)
- moved SY1 2.54 mm to (9.37, 1.75)
- moved JP3 2.54 mm to (5.08, 47.0)
- moved JP4 2.54 mm to (5.08, 3.81)
- moved LED1 0.48 mm to (71.1, 8.10)
- moved R2 0.16 mm to (69.2, 7.78)
Routing:
- net N$9: track 3.05 -> 11.1 mm
- net N$6: track 3.05 -> 5.40 mm
- net VALVE_POT: track 69.1 -> 71.1 mm
- net INDEX_OUT: track 21.7 -> 19.8 mm
- net INDEX_IN: track 10.3 -> 8.65 mm
- net +5V: track 239.6 -> 240.8 mm
Other:
- board size 91.4 x 50.8 mm -> 82.5 x 50.8 mm
- board text added: "FBACK"
- board text added: "INDEX"
- board text removed: "INDEX FB"

Commit message: foo
Parts:
- removed S1: Reset, freetronics-master-v1:TACTILE_SWITCH_SMD_2PIN_TINY
- added S2: Reset, freetronics-luke:FSMSM
Connections:
- net !RESET: now also S2.1; no longer S1.2
- net GND: now also S2.2; no longer S1.1
Routing:
- net GND: vias 4 -> 6
Changed lines of the file:
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@@
 <text x="11.7475" y="2.06375" size="0.8128" layer="21" ratio="15">R2020 Servo Controller</text>
 <text x="13.335" y="0.635" size="0.8128" layer="21" ratio="15">Luke Weston, 2013</text>
-<text x="21.59" y="6.82625" size="0.8128" layer="21" ratio="15">Reset</text>
+<text x="18.57375" y="6.985" size="0.8128" layer="21" ratio="15">Reset</text>
 <text x="12.3825" y="47.14875" size="0.8128" layer="21" ratio="15">Power</text>
 <text x="82.55" y="32.0675" size="0.8128" layer="21" ratio="15" rot="SR270">INDEX</text>
@@
 <element name="R18" library="freetronics-master-v1" package="0603" value="120Ω" x="16.51" y="9.8425" smashed="yes" rot="R90">
 <attribute name="PACKAGE" value="0603" x="106.68" y="59.3725" size="1.778" layer="27" rot="R90" display="off"/>
-<attribute name="NAME" x="16.9545" y="6.25475" size="0.8128" layer="25" font="vector" ratio="15" rot="R90"/>
-<attribute name="VALUE" x="16.98625" y="5.55625" size="0.8128" layer="27" font="vector" ratio="15" rot="R90"/>
+<attribute name="NAME" x="13.716" y="8.60425" size="0.8128" layer="25" font="vector" ratio="15"/>
+<attribute name="VALUE" x="13.0175" y="8.5725" size="0.8128" layer="27" font="vector" ratio="15"/>
 </element>
 <element name="R21" library="freetronics-master-v1" package="0603" value="10kΩ" x="24.257" y="19.05" smashed="yes">
@@
 <element name="R19" library="freetronics-master-v1" package="0603" value="100Ω" x="18.415" y="9.8425" smashed="yes" rot="R270">
 <attribute name="PACKAGE" value="0603" x="-71.755" y="-47.3075" size="1.778" layer="27" rot="R270" display="off"/>
-<attribute name="NAME" x="18.8595" y="6.4135" size="0.8128" layer="25" font="vector" ratio="15" rot="R90"/>
-<attribute name="VALUE" x="18.90395" y="5.49275" size="0.8128" layer="27" font="vector" ratio="15" rot="R90"/>
+<attribute name="NAME" x="17.36725" y="7.65175" size="0.8128" layer="25" font="vector" ratio="15"/>
+<attribute name="VALUE" x="16.92275" y="7.6073" size="0.8128" layer="27" font="vector" ratio="15"/>
 </element>
 <element name="R20" library="freetronics-master-v1" package="0603" value="100Ω" x="19.685" y="17.78" smashed="yes" rot="R90">
@@
 <element name="R15" library="freetronics-master-v1" package="0603" value="10kΩ" x="45.56125" y="30.32125" smashed="yes" rot="R270">
 <attribute name="PACKAGE" value="0603" x="45.56125" y="30.32125" size="1.778" layer="27" rot="R270" display="off"/>
-<attribute name="NAME" x="42.926" y="29.87675" size="0.8128" layer="25" font="vector" ratio="15"/>
-<attribute name="VALUE" x="47.0027" y="28.829" size="0.8128" layer="27" font="vector" ratio="15" rot="R90"/>
+<attribute name="NAME" x="44.8945" y="29.2735" size="0.8128" layer="25" font="vector" ratio="15" rot="R90"/>
+<attribute name="VALUE" x="44.93895" y="28.829" size="0.8128" layer="27" font="vector" ratio="15" rot="R90"/>
 </element>
 <element name="R14" library="freetronics-master-v1" package="0603" value="10kΩ" x="33.17875" y="2.54" smashed="yes">
@@
 <attribute name="VALUE" x="56.4515" y="29.8323" size="0.8128" layer="27" font="vector" ratio="15"/>
 </element>
-<element name="S1" library="freetronics-master-v1" package="TACTILE_SWITCH_SMD_2PIN_TINY" value="Reset" x="23.33625" y="5.08" smashed="yes"/>
 <element name="J13" library="freetronics-master-v1" package="1X05" value="Encoder" x="69.85" y="17.78" smashed="yes" rot="R90">
 <attribute name="NAME" x="68.8213" y="29.61005" size="0.8128" layer="25" ratio="15"/>
@@
 <attribute name="NAME" x="12.92225" y="45.11675" size="0.8128" layer="25" font="vector" ratio="15"/>
 <attribute name="VALUE" x="12.954" y="45.0723" size="0.8128" layer="27" font="vector" ratio="15"/>
+</element>
+<element name="S2" library="freetronics-luke" package="FSMSM" value="Reset" x="20.32" y="5.08" smashed="yes" rot="R180">
+<attribute name="PACKAGE" value="FSMSM" x="20.32" y="5.08" size="0.8128" layer="27" ratio="15" rot="R180" display="off"/>
+<attribute name="NAME" x="13.81125" y="7.14375" size="0.8128" layer="25" ratio="15"/>
+<attribute name="VALUE" x="13.81125" y="6.19125" size="0.8128" layer="27" ratio="15"/>
 </element>
 </elements>
@@
 <contactref element="LED4" pad="C"/>
 <polygon width="0.4064" layer="1">
-<vertex x="-2.54" y="52.07"/>
-<vertex x="91.44" y="52.07"/>
-<vertex x="91.44" y="-1.27"/>
-<vertex x="-2.54" y="-1.27"/>
+<vertex x="0" y="52.07"/>
+<vertex x="85.09" y="52.07"/>
+<vertex x="85.09" y="-1.27"/>
+<vertex x="0" y="-1.27"/>
 </polygon>
 <contactref element="LED2" pad="C"/>
-<contactref element="S1" pad="1"/>
 <contactref element="IC3" pad="5"/>
 <contactref element="IC3" pad="PAD"/>
@@
 <wire x1="36.195" y1="33.02" x2="36.195" y2="34.29" width="0.4064" layer="1"/>
 <polygon width="0.4064" layer="16">
-<vertex x="-2.54" y="52.07"/>
-<vertex x="91.44" y="52.07"/>
-<vertex x="91.44" y="-1.27"/>
-<vertex x="-2.54" y="-1.27"/>
+<vertex x="0" y="52.07"/>
+<vertex x="85.09" y="52.07"/>
+<vertex x="85.09" y="-1.27"/>
+<vertex x="0" y="-1.27"/>
 </polygon>
 <wire x1="35.56" y1="30.42" x2="35.56" y2="32.385" width="0.4064" layer="1"/>
@@
 <contactref element="C5" pad="1"/>
 <contactref element="LED5" pad="C"/>
+<contactref element="S2" pad="2"/>
+<via x="33.02" y="12.7" extent="1-16" drill="0.4"/>
+<via x="43.18" y="35.56" extent="1-16" drill="0.4"/>
 </signal>
 <signal name="+5V">
@@
 <wire x1="33.02" y1="21.59" x2="34.29" y2="21.59" width="0.6096" layer="16"/>
 <wire x1="34.29" y1="21.59" x2="38.1" y2="25.4" width="0.6096" layer="16"/>
-<contactref element="S1" pad="2"/>
 <contactref element="C4" pad="1"/>
 <wire x1="48.66" y1="5.988" x2="47.752" y2="5.08" width="0.6096" layer="1"/>
-<wire x1="25.38625" y1="5.08" x2="27.14625" y2="5.08" width="0.8128" layer="1"/>
 <via x="27.14625" y="5.08" extent="1-16" drill="0.4"/>
 <wire x1="27.14625" y1="5.08" x2="24.765" y2="7.46125" width="0.6096" layer="16"/>
@@
 <wire x1="31.75" y1="18.7579" x2="31.75" y2="20.32" width="0.6096" layer="1"/>
 <wire x1="31.75" y1="20.32" x2="33.02" y2="21.59" width="0.6096" layer="1"/>
+<contactref element="S2" pad="1"/>
+<wire x1="24.9174" y1="5.08" x2="27.14625" y2="5.08" width="0.6096" layer="1"/>
 </signal>
 <signal name="!CAN_CS">

Commit message: foo
Parts:
- renumbered S2 to S1
Changed lines of the file:
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@@
 <attribute name="VALUE" x="12.954" y="45.0723" size="0.8128" layer="27" font="vector" ratio="15"/>
 </element>
-<element name="S2" library="freetronics-luke" package="FSMSM" value="Reset" x="20.32" y="5.08" smashed="yes" rot="R180">
+<element name="S1" library="freetronics-luke" package="FSMSM" value="Reset" x="20.32" y="5.08" smashed="yes" rot="R180">
 <attribute name="PACKAGE" value="FSMSM" x="20.32" y="5.08" size="0.8128" layer="27" ratio="15" rot="R180" display="off"/>
 <attribute name="NAME" x="13.81125" y="7.14375" size="0.8128" layer="25" ratio="15"/>
@@
 <contactref element="C5" pad="1"/>
 <contactref element="LED5" pad="C"/>
-<contactref element="S2" pad="2"/>
+<contactref element="S1" pad="2"/>
 <via x="33.02" y="12.7" extent="1-16" drill="0.4"/>
 <via x="43.18" y="35.56" extent="1-16" drill="0.4"/>
@@
 <wire x1="31.75" y1="18.7579" x2="31.75" y2="20.32" width="0.6096" layer="1"/>
 <wire x1="31.75" y1="20.32" x2="33.02" y2="21.59" width="0.6096" layer="1"/>
-<contactref element="S2" pad="1"/>
+<contactref element="S1" pad="1"/>
 <wire x1="24.9174" y1="5.08" x2="27.14625" y2="5.08" width="0.6096" layer="1"/>
 </signal>
