File: R2020Interface.sch (EAGLE design)
At the start: 83 parts, among them IC1 ATmega328-AU, IC2 RT8289, IC3 LM5010SD, IC4 MCP2515-I/SO, IC5 MCP2551, J1 ISP, J10 Position feedback pot, J11 CAN Terminate, J12 AS5040, J13 Encoder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

Commit message: foo
Parts:
- removed S1: Reset, freetronics-master-v1:TAC_SWITCH_2PIN
- added S2: Reset, freetronics-luke:FSMSM
Connections:
- net !RESET: now also S2.1; no longer S1.S
- net GND: now also S2.2; no longer S1.P
Changed lines of the file:
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@@
 </part>
 <part name="U$46" library="freetronics-luke" deviceset="+5V" device=""/>
-<part name="S1" library="freetronics-master-v1" deviceset="TAC_SWITCH_2PIN" device="" value="Reset"/>
 <part name="U$47" library="freetronics-luke" deviceset="GND" device=""/>
 <part name="J13" library="freetronics-master-v1" deviceset="M05" device="PTH" value="Encoder"/>
@@
 </part>
 <part name="U$60" library="freetronics-luke" deviceset="+5V" device=""/>
+<part name="S2" library="freetronics-luke" deviceset="FSMSM" device="" value="Reset">
+<attribute name="PACKAGE" value="FSMSM"/>
+</part>
 </parts>
 <sheets>
@@
 </instance>
 <instance part="U$46" gate="G$1" x="231.14" y="322.58" rot="MR0"/>
-<instance part="S1" gate="1" x="167.64" y="424.18" smashed="yes" rot="R90">
-<attribute name="NAME" x="160.02" y="419.1" size="1.27" layer="95"/>
-<attribute name="VALUE" x="160.02" y="416.56" size="1.27" layer="96"/>
-</instance>
 <instance part="U$47" gate="G$1" x="167.64" y="414.02"/>
 <instance part="J13" gate="G$1" x="203.2" y="91.44" smashed="yes" rot="R180">
@@
 </instance>
 <instance part="U$60" gate="G$1" x="233.68" y="76.2"/>
+<instance part="S2" gate="G$1" x="167.64" y="424.18" smashed="yes" rot="R270">
+<attribute name="PACKAGE" x="160.02" y="421.64" size="1.27" layer="96"/>
+<attribute name="NAME" x="160.02" y="426.72" size="1.27" layer="95"/>
+<attribute name="VALUE" x="160.02" y="424.18" size="1.27" layer="96"/>
+</instance>
 </instances>
 <busses>
@@
 </segment>
 <segment>
-<pinref part="S1" gate="1" pin="P"/>
 <pinref part="U$47" gate="G$1" pin="GND"/>
 <wire x1="167.64" y1="416.56" x2="167.64" y2="419.1" width="0.1524" layer="91"/>
+<pinref part="S2" gate="G$1" pin="2"/>
 </segment>
 <segment>
@@
 <junction x="167.64" y="439.42"/>
 <label x="160.02" y="439.674" size="1.27" layer="95"/>
-<pinref part="S1" gate="1" pin="S"/>
-<wire x1="167.64" y1="429.26" x2="167.64" y2="439.42" width="0.1524" layer="91"/>
+<wire x1="167.64" y1="429.26" x2="167.64" y2="436.88" width="0.1524" layer="91"/>
 <pinref part="C5" gate="G$1" pin="2"/>
-<wire x1="175.26" y1="426.72" x2="175.26" y2="431.8" width="0.1524" layer="91"/>
-<wire x1="175.26" y1="431.8" x2="167.64" y2="439.42" width="0.1524" layer="91"/>
-</segment>
-<segment>
+<wire x1="167.64" y1="436.88" x2="167.64" y2="439.42" width="0.1524" layer="91"/>
+<pinref part="S2" gate="G$1" pin="1"/>
+<wire x1="175.26" y1="426.72" x2="175.26" y2="429.26" width="0.1524" layer="91"/>
+<wire x1="175.26" y1="429.26" x2="167.64" y2="436.88" width="0.1524" layer="91"/>
+<junction x="167.64" y="436.88"/>
+</segment>
+<segment>

Commit message: foo
Parts:
- renumbered S2 to S1
Changed lines of the file:
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@@
 </part>
 <part name="U$60" library="freetronics-luke" deviceset="+5V" device=""/>
-<part name="S2" library="freetronics-luke" deviceset="FSMSM" device="" value="Reset">
+<part name="S1" library="freetronics-luke" deviceset="FSMSM" device="" value="Reset">
 <attribute name="PACKAGE" value="FSMSM"/>
 </part>
@@
 </instance>
 <instance part="U$60" gate="G$1" x="233.68" y="76.2"/>
-<instance part="S2" gate="G$1" x="167.64" y="424.18" smashed="yes" rot="R270">
+<instance part="S1" gate="G$1" x="167.64" y="424.18" smashed="yes" rot="R270">
 <attribute name="PACKAGE" x="160.02" y="421.64" size="1.27" layer="96"/>
 <attribute name="NAME" x="160.02" y="426.72" size="1.27" layer="95"/>
@@
 <pinref part="U$47" gate="G$1" pin="GND"/>
 <wire x1="167.64" y1="416.56" x2="167.64" y2="419.1" width="0.1524" layer="91"/>
-<pinref part="S2" gate="G$1" pin="2"/>
+<pinref part="S1" gate="G$1" pin="2"/>
 </segment>
 <segment>
@@
 <pinref part="C5" gate="G$1" pin="2"/>
 <wire x1="167.64" y1="436.88" x2="167.64" y2="439.42" width="0.1524" layer="91"/>
-<pinref part="S2" gate="G$1" pin="1"/>
+<pinref part="S1" gate="G$1" pin="1"/>
 <wire x1="175.26" y1="426.72" x2="175.26" y2="429.26" width="0.1524" layer="91"/>
 <wire x1="175.26" y1="429.26" x2="167.64" y2="436.88" width="0.1524" layer="91"/>
